File: pcb/WeAct-STM32G474.kicad_pcb (KiCad board)
At the start: 2 copper layers, 50 x 40 mm, 36 parts, among them J3 P1, J4 P2, U1 AMS1117-3.3, U2 SRV05-4, U3 STM32G474CBTx, Y1 X_24MHZ

Commit message: Complete PCB
Parts:
- moved C4 4.29 mm to (142.7, 98.4), turned to 90 degrees
- moved D3 0.80 mm to (120.8, 91.7)
- moved R6 0.80 mm to (121.7, 94.7)
- moved C2 0.20 mm to (124.2, 96.8)
Connections:
- D4 pad 1: VB -> +3V3
- D4 pad 2: +3V3 -> VB
- J4 pad 10: PB1 -> PB2
- J4 pad 12: unconnected-(J4-Pin_12-Pad12) -> PB0
- J4 pad 22: PC13 -> PC15
- J4 pad 24: PC15 -> PC13
- J4 pad 5: PB10 -> PB11
- J4 pad 6: PB11 -> PB10
- J4 pad 7: PB2 -> VREF
- J4 pad 8: VREF -> unconnected-(J4-Pin_8-Pad8)
- J4 pad 9: PB0 -> PB1
Routing:
- net NRST: track 0.00 -> 57.1 mm
- net GND: track 53.5 -> 83.9 mm, vias 10 -> 13
- net PB8_BOOT0: track 37.9 -> 67.0 mm
- net PB11: track 0.00 -> 22.6 mm, vias 0 -> 1
- net PB10: track 0.00 -> 21.0 mm, vias 0 -> 1
- net PC13: track 8.45 -> 28.2 mm, vias 0 -> 1
- net PB12: track 0.00 -> 19.6 mm, vias 0 -> 1
- net PB2: track 0.00 -> 19.1 mm, vias 0 -> 1
- net PB0: track 0.00 -> 18.3 mm, vias 0 -> 1
- net PB14: track 0.00 -> 18.1 mm, vias 0 -> 1
- net PC15: track 0.00 -> 17.6 mm, vias 0 -> 1
- net PA6: track 0.00 -> 17.4 mm, vias 0 -> 1
- net PA0: track 0.00 -> 15.9 mm, vias 0 -> 1
- net PC14: track 0.00 -> 15.9 mm, vias 0 -> 1
- net PB13: track 0.00 -> 15.8 mm, vias 0 -> 1
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
Commit message: pcb design phase 1
Parts:
- removed the C14 at (142.6, 104.2)
- removed C15, C17, C6: C_100NF_0603, Capacitor_SMD:C_0603_1608Metric_Pad1.08x0.95mm_HandSolder
- removed C16: C_1UF_0603, Capacitor_SMD:C_0603_1608Metric_Pad1.08x0.95mm_HandSolder
- added C10: C_100NF_0603, Capacitor_SMD:C_0603_1608Metric, F.Cu at (135.3, 104.2)
- added C7: C_100NF_0603, Capacitor_SMD:C_0603_1608Metric, F.Cu at (137.0, 104.2)
- added C9: C_1UF_0603, Capacitor_SMD:C_0603_1608Metric, F.Cu at (132.9, 105.2)
- added REF**: MountingHole_2.1mm, MountingHole:MountingHole_2.1mm, F.Cu at (121.0, 116.0)
- added REF**: MountingHole_2.1mm, MountingHole:MountingHole_2.1mm, F.Cu at (167.0, 116.0)
- added REF**: MountingHole_2.1mm, MountingHole:MountingHole_2.1mm, F.Cu at (121.0, 80.0)
- added REF**: MountingHole_2.1mm, MountingHole:MountingHole_2.1mm, F.Cu at (167.0, 80.0)
- C1: footprint Capacitor_SMD:C_0805_2012Metric_Pad1.18x1.45mm_HandSolder -> Capacitor_SMD:C_0805_2012Metric
- C12: value C_100NF_0603 -> C_20PF_0603; footprint Capacitor_SMD:C_0603_1608Metric_Pad1.08x0.95mm_HandSolder -> Capacitor_SMD:C_0603_1608Metric
- C13: value C_20PF_0603 -> C_100NF_0603
- C14: renamed from C10; footprint Capacitor_SMD:C_0603_1608Metric_Pad1.08x0.95mm_HandSolder -> Capacitor_SMD:C_0603_1608Metric
- C2: value C_100NF_0603 -> C_10UF_0805; footprint Capacitor_SMD:C_0603_1608Metric_Pad1.08x0.95mm_HandSolder -> Capacitor_SMD:C_0805_2012Metric
- C3: value C_10UF_0805 -> C_1UF_0805; footprint Capacitor_SMD:C_0805_2012Metric_Pad1.18x1.45mm_HandSolder -> Capacitor_SMD:C_0603_1608Metric
- C4: value C_1UF_0805 -> C_100NF_0603; footprint Capacitor_SMD:C_0805_2012Metric_Pad1.18x1.45mm_HandSolder -> Capacitor_SMD:C_0603_1608Metric
- C5: footprint Capacitor_SMD:C_0603_1608Metric_Pad1.08x0.95mm_HandSolder -> Capacitor_SMD:C_0603_1608Metric
- C8: value C_100NF_0603 -> C_1UF_0603; footprint Capacitor_SMD:C_0603_1608Metric_Pad1.08x0.95mm_HandSolder -> Capacitor_SMD:C_0603_1608Metric
- R1, R2, R3: footprint Resistor_SMD:R_0603_1608Metric_Pad0.98x0.95mm_HandSolder -> Resistor_SMD:R_0603_1608Metric
- R4: renamed from R5; footprint Resistor_SMD:R_0603_1608Metric_Pad0.98x0.95mm_HandSolder -> Resistor_SMD:R_0603_1608Metric
- R5: renamed from R6; footprint Resistor_SMD:R_0603_1608Metric_Pad0.98x0.95mm_HandSolder -> Resistor_SMD:R_0603_1608Metric
- R6: renamed from R4; footprint Resistor_SMD:R_0603_1608Metric_Pad0.98x0.95mm_HandSolder -> Resistor_SMD:R_0603_1608Metric
- moved C2 23.2 mm to (147.2, 99.8), turned to 90 degrees
- moved C3 18.5 mm to (129.9, 92.8), turned to 180 degrees
- moved D1 16.5 mm to (123.7, 92.6)
- moved C12 13.9 mm to (123.9, 101.5), turned to 180 degrees
- moved D4 13.8 mm to (123.8, 105.2), turned to 180 degrees
- moved C5 13.4 mm to (140.3, 101.7), turned to 0 degrees
- moved R4 12.8 mm to (153.2, 96.3)
- moved D3 12.7 mm to (149.9, 96.3)
- moved C13 10.8 mm to (127.2, 94.3), turned to 180 degrees
- moved R5 8.96 mm to (123.8, 103.4)
- moved C4 6.99 mm to (140.0, 92.0)
- moved R6 6.00 mm to (161.0, 90.4), turned to 0 degrees
- moved C8 5.35 mm to (139.4, 105.0), turned to 180 degrees
- moved C11 5.14 mm to (123.9, 95.5), turned to 180 degrees
- moved Y1 4.67 mm to (123.7, 98.5), turned to -90 degrees
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- renumbered BOOT1 to BOOT, D4 to D1, D1 to D2, D2 to D3, D3 to D4, J3 to J1, J4 to J2, J1 to J3, NRST1 to NRST, U3 to U2, U2 to U3
Connections:
- C12 pad 1: VREF -> Net-(U2-PF1)
- C13 pad 1: Net-(U3-PF1) -> VBAT
- J1 pad 1: +5V -> +3V3
- J1 pad 2: +5V -> +3V3
- J2 pad 1: +3V3 -> +5V
- J2 pad 2: +3V3 -> +5V
- U2 pad 6: Net-(U3-PF1) -> Net-(U2-PF1)
- Y1 pad 3: Net-(U3-PF1) -> Net-(U2-PF1)
Routing:
- net +5V: track 34.7 -> 5.49 mm, vias 1 -> 0
- net NRST: track 57.1 -> 32.7 mm
- net PB11: track 22.6 -> 0.00 mm, vias 1 -> 0
- net PB10: track 21.0 -> 0.00 mm, vias 1 -> 0
- net PA11: track 51.8 -> 31.5 mm
- net PA12: track 49.5 -> 29.6 mm
- net PB2: track 19.1 -> 0.00 mm, vias 1 -> 0
- net PB0: track 18.3 -> 0.00 mm, vias 1 -> 0
- net PA6: track 17.4 -> 0.00 mm, vias 1 -> 0
- net PB1: track 15.7 -> 0.00 mm, vias 1 -> 0
- net PA7: track 15.2 -> 0.00 mm, vias 1 -> 0
- net VB: track 3.74 -> 17.1 mm, vias 0 -> 1
- net PA5: track 13.1 -> 0.00 mm, vias 1 -> 0
- net VREF: track 19.7 -> 6.80 mm, vias 1 -> 0
- net VBAT: track 18.5 -> 7.33 mm
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
Commit message: pcb design phase 2
Parts:
- moved C10 0.25 mm to (135.3, 104.5)
- moved C7 0.25 mm to (137.0, 104.5)
- moved C8 0.25 mm to (139.4, 105.3)
- moved C9 0.25 mm to (132.9, 105.4)
- moved FB1 0.25 mm to (139.4, 103.7)
- moved FB2 0.25 mm to (132.9, 103.7)
- turned R5 to 180 degrees
Routing:
- net PB10: track 0.00 -> 17.2 mm, vias 0 -> 1
- net PB2: track 0.00 -> 16.9 mm, vias 0 -> 1
- net PA12: track 29.6 -> 45.4 mm
- net PB0: track 0.00 -> 15.3 mm, vias 0 -> 1
- net PB11: track 0.00 -> 15.2 mm, vias 0 -> 1
- net PA11: track 31.5 -> 46.3 mm
- net PA6: track 0.00 -> 13.8 mm, vias 0 -> 1
- net PB1: track 0.00 -> 12.9 mm, vias 0 -> 1
- net PA7: track 0.00 -> 11.4 mm, vias 0 -> 1
- net VREF: track 6.80 -> 17.8 mm, vias 0 -> 1
- net +5V: track 5.49 -> 16.4 mm, vias 0 -> 1
- net PA5: track 0.00 -> 10.5 mm, vias 0 -> 1
- net PC13: track 22.4 -> 32.6 mm
- net GND: track 86.7 -> 93.2 mm, vias 13 -> 15
- net +3V3: track 7.10 -> 9.03 mm
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
Commit message: pcb design phase 3
Routing:
- net GND: track 93.2 -> 93.9 mm, vias 15 -> 16
- net Net-(J3-CC2): track 7.95 -> 7.29 mm
- net PA12: track 45.4 -> 46.1 mm

Commit message: pcb design phase 4
Parts:
- moved C14 5.64 mm to (166.3, 106.9)
- moved D2 5.55 mm to (158.1, 101.4), turned to 90 degrees
- moved C1 4.52 mm to (146.5, 103.4), turned to 90 degrees
- moved R3 2.81 mm to (163.5, 106.0), turned to -90 degrees
- moved D3 0.86 mm to (149.2, 96.8)
- moved R4 0.86 mm to (152.5, 96.8)
- moved U1 0.86 mm to (152.3, 101.5)
- moved C2 0.73 mm to (146.5, 99.6)
- moved C13 0.06 mm to (127.2, 94.3)
- turned BOOT to 180 degrees
- turned NRST to 0 degrees
Routing:
- net NRST: track 33.2 -> 70.2 mm
- net VBUS: track 26.1 -> 20.4 mm
- net +5V: track 16.4 -> 20.8 mm
- net +3V3: track 9.03 -> 13.1 mm
- net PB8_BOOT0: track 67.3 -> 63.6 mm, vias 0 -> 1
- net GND: track 93.9 -> 92.1 mm, vias 16 -> 17
- net VB: track 18.5 -> 17.2 mm
- net PB10: track 17.2 -> 16.1 mm

Commit message: pcb design complete
Parts:
- D1: footprint Package_TO_SOT_SMD:SOT-323_SC-70 -> Package_TO_SOT_SMD:TSOT-23
- D2: value ~ -> DFLS140; footprint Diode_SMD:D_SOD-123 -> Diode_SMD:D_PowerDI-123
- FB1, FB2: value FB_0603 -> FB_0805; footprint Inductor_SMD:L_0603_1608Metric -> Inductor_SMD:L_0805_2012Metric
- R1, R2: value R_5.1K_0805 -> R_5.1K_0603
- R3, R6: value R_10K_0805 -> R_10K_0603
- R4, R5: value R_220_0805 -> R_220_0603
- Y1: footprint Crystal:Crystal_SMD_3225-4Pin_3.2x2.5mm -> Crystal:Crystal_SMD_2016-4Pin_2.0x1.6mm
- moved D1 0.85 mm to (123.4, 91.8)
- moved FB2 0.76 mm to (132.3, 104.2)
- moved C8 0.75 mm to (139.1, 106.0)
- moved C10 0.66 mm to (135.0, 105.1)
- moved C7 0.66 mm to (136.7, 105.1)
- moved C9 0.66 mm to (132.6, 106.0)
- moved FB1 0.50 mm to (139.4, 104.2)
- renumbered BOOT to BOOT1, NRST to NRST1
Connections:
- J2 pad 10: PB2 -> PB1
- J2 pad 11: PA7 -> PB0
- J2 pad 12: PB0 -> PA7
- J2 pad 13: PA5 -> PA6
- J2 pad 14: PA6 -> PA5
- J2 pad 9: PB1 -> PB2
Routing:
- net PB1: track 12.8 -> 16.8 mm
- net PA7: track 11.3 -> 15.1 mm
- net PA5: track 10.6 -> 14.3 mm
- net PB2: track 17.0 -> 14.0 mm
- net PB0: track 15.4 -> 12.7 mm
- net PA11: track 46.3 -> 48.8 mm
- net PA6: track 13.9 -> 11.4 mm
- net +3V3: track 13.1 -> 10.8 mm
- net NRST: track 70.2 -> 68.1 mm
- net PA2: track 20.8 -> 18.7 mm
- net PA0: track 21.1 -> 19.0 mm
- net PA4: track 21.2 -> 19.2 mm
- net PA3: track 17.6 -> 15.6 mm
- net PB12: track 20.6 -> 22.6 mm
- net Net-(J3-CC2): track 7.32 -> 9.23 mm
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
Commit message: pcb design update 1
Parts:
- C11, C12: value C_20PF_0603 -> C_10PF_0402; footprint Capacitor_SMD:C_0603_1608Metric -> Capacitor_SMD:C_0402_1005Metric
- moved C12 1.17 mm to (124.7, 100.7)
- moved Y1 1.01 mm to (124.7, 98.4)
- moved C11 0.97 mm to (124.7, 96.1)
- renumbered BOOT1 to BOOT, NRST1 to NRST
Routing:
- net Net-(U2-PF1): track 10.7 -> 8.77 mm
- net Net-(U2-PF0): track 9.71 -> 8.09 mm
- net +5V: track 21.6 -> 22.4 mm, vias 1 -> 2
- net GND: track 90.6 -> 89.9 mm
