File: pcb/WeAct-STM32G474.kicad_sch (KiCad schematic)
At the start: 36 parts, among them J3 P1, J4 P2, U1 AMS1117-3.3, U2 SRV05-4, U3 STM32G474CBTx, Y1 X_24MHZ

Commit message: Complete PCB
Connections:
- net +3V3: now also D4.1; no longer D4.2
- net PB0: now also J4.12 (Pin_12); no longer J4.9 (Pin_9)
- net PB1: now also J4.9 (Pin_9); no longer J4.10 (Pin_10)
- net PB10: now also J4.6 (Pin_6); no longer J4.5 (Pin_5)
- net PB11: now also J4.5 (Pin_5); no longer J4.6 (Pin_6)
- net PB2: now also J4.10 (Pin_10); no longer J4.7 (Pin_7)
- net PC13: now also J4.24 (Pin_24); no longer J4.22 (Pin_22)
- net PC15: now also J4.22 (Pin_22); no longer J4.24 (Pin_24)
- net VB: now also D4.2; no longer D4.1
- net VREF: now also J4.7 (Pin_7); no longer J4.8 (Pin_8)
- no-connect marks 6 -> 5

Commit message: pcb design phase 1
Parts:
- removed C14: C_1UF_0805, Capacitor_SMD:C_0805_2012Metric_Pad1.18x1.45mm_HandSolder, symbol stm32world:C_1UF_0603
- removed C15, C2: C_100NF_0603, Capacitor_SMD:C_0603_1608Metric_Pad1.08x0.95mm_HandSolder, symbol stm32world:C_100NF_0603
- added C9: C_1UF_0603, Capacitor_SMD:C_0603_1608Metric, symbol stm32world:C_1UF_0603
- C1: footprint Capacitor_SMD:C_0805_2012Metric_Pad1.18x1.45mm_HandSolder -> Capacitor_SMD:C_0805_2012Metric
- C10: renamed from C12; footprint Capacitor_SMD:C_0603_1608Metric_Pad1.08x0.95mm_HandSolder -> Capacitor_SMD:C_0603_1608Metric
- C13: renamed from C17; footprint Capacitor_SMD:C_0603_1608Metric_Pad1.08x0.95mm_HandSolder -> Capacitor_SMD:C_0603_1608Metric
- C14: renamed from C10; footprint Capacitor_SMD:C_0603_1608Metric_Pad1.08x0.95mm_HandSolder -> Capacitor_SMD:C_0603_1608Metric
- C2: renamed from C3; footprint Capacitor_SMD:C_0805_2012Metric_Pad1.18x1.45mm_HandSolder -> Capacitor_SMD:C_0805_2012Metric
- C3: renamed from C4; footprint Capacitor_SMD:C_0805_2012Metric_Pad1.18x1.45mm_HandSolder -> Capacitor_SMD:C_0603_1608Metric
- C4: renamed from C5; footprint Capacitor_SMD:C_0603_1608Metric_Pad1.08x0.95mm_HandSolder -> Capacitor_SMD:C_0603_1608Metric
- C5: renamed from C6; footprint Capacitor_SMD:C_0603_1608Metric_Pad1.08x0.95mm_HandSolder -> Capacitor_SMD:C_0603_1608Metric
- C7: renamed from C8; footprint Capacitor_SMD:C_0603_1608Metric_Pad1.08x0.95mm_HandSolder -> Capacitor_SMD:C_0603_1608Metric
- C8: renamed from C16; footprint Capacitor_SMD:C_0603_1608Metric_Pad1.08x0.95mm_HandSolder -> Capacitor_SMD:C_0603_1608Metric
- R1, R2, R3: footprint Resistor_SMD:R_0603_1608Metric_Pad0.98x0.95mm_HandSolder -> Resistor_SMD:R_0603_1608Metric
- R4: renamed from R5; footprint Resistor_SMD:R_0603_1608Metric_Pad0.98x0.95mm_HandSolder -> Resistor_SMD:R_0603_1608Metric
- R5: renamed from R6; footprint Resistor_SMD:R_0603_1608Metric_Pad0.98x0.95mm_HandSolder -> Resistor_SMD:R_0603_1608Metric
- R6: renamed from R4; footprint Resistor_SMD:R_0603_1608Metric_Pad0.98x0.95mm_HandSolder -> Resistor_SMD:R_0603_1608Metric
- renumbered C13 to C12, D4 to D1, D1 to D2, D2 to D3, D3 to D4, J3 to J1, J4 to J2, J1 to J3, U3 to U2, U2 to U3
Connections:
- net +3V3: now also J1.1 (Pin_1), J1.2 (Pin_2); no longer J2.1 (Pin_1), J2.2 (Pin_2)
- net +5V: now also J2.1 (Pin_1), J2.2 (Pin_2); no longer J1.1 (Pin_1), J1.2 (Pin_2)
- net GND: now also C9.2
- net VREF: now also C9.1
- no-connect marks 5 -> 6
Other:
- moved on the sheet: C10, C7, C8

Commit message: pcb design complete
Parts:
- C11, C12: Display 20pF -> 10pF
- D1: footprint Package_TO_SOT_SMD:SOT-323_SC-70 -> Package_TO_SOT_SMD:TSOT-23
- D2: value ~ -> DFLS140; footprint Diode_SMD:D_SOD-123 -> Diode_SMD:D_PowerDI-123
- FB1, FB2: value FB_0603 -> FB_0805; footprint Inductor_SMD:L_0603_1608Metric -> Inductor_SMD:L_0805_2012Metric
- R1, R2: value R_5.1K_0805 -> R_5.1K_0603
- R3, R6: value R_10K_0805 -> R_10K_0603
- R4, R5: value R_220_0805 -> R_220_0603
- Y1: footprint Crystal:Crystal_SMD_3225-4Pin_3.2x2.5mm -> Crystal:Crystal_SMD_2016-4Pin_2.0x1.6mm
Connections:
- net PA5: now also J2.14 (Pin_14); no longer J2.13 (Pin_13)
- net PA6: now also J2.13 (Pin_13); no longer J2.14 (Pin_14)
- net PA7: now also J2.12 (Pin_12); no longer J2.11 (Pin_11)
- net PB0: now also J2.11 (Pin_11); no longer J2.12 (Pin_12)
- net PB1: now also J2.10 (Pin_10); no longer J2.9 (Pin_9)
- net PB2: now also J2.9 (Pin_9); no longer J2.10 (Pin_10)
Changed lines of the file:
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@@
 	(wire
 		(pts
+			(xy 254 105.41) (xy 256.54 105.41)
+		)
+		(stroke
+			(width 0)
+			(type default)
+		)
+	)
+	(wire
+		(pts
 			(xy 62.23 175.26) (xy 58.42 175.26)
 		)
@@
 	(wire
 		(pts
-			(xy 254 105.41) (xy 256.54 105.41)
+			(xy 238.76 67.31) (xy 241.3 67.31)
 		)
 		(stroke
@@
 	(wire
 		(pts
-			(xy 238.76 67.31) (xy 241.3 67.31)
+			(xy 238.76 46.99) (xy 241.3 46.99)
 		)
 		(stroke
@@
 	(wire
 		(pts
-			(xy 238.76 46.99) (xy 241.3 46.99)
+			(xy 66.04 128.27) (xy 66.04 130.81)
 		)
 		(stroke
@@
 	(wire
 		(pts
-			(xy 66.04 128.27) (xy 66.04 130.81)
+			(xy 198.12 90.17) (xy 201.93 90.17)
 		)
 		(stroke
@@
 	(wire
 		(pts
-			(xy 198.12 90.17) (xy 201.93 90.17)
+			(xy 121.92 90.17) (xy 121.92 92.71)
 		)
 		(stroke
@@
 	(wire
 		(pts
-			(xy 121.92 90.17) (xy 121.92 92.71)
+			(xy 254 113.03) (xy 256.54 113.03)
 		)
 		(stroke
@@
 	(wire
 		(pts
-			(xy 254 113.03) (xy 256.54 113.03)
+			(xy 254 100.33) (xy 256.54 100.33)
 		)
 		(stroke
@@
 	(wire
 		(pts
-			(xy 238.76 102.87) (xy 241.3 102.87)
+			(xy 55.88 135.89) (xy 55.88 138.43)
 		)
 		(stroke
@@
 	(wire
 		(pts
-			(xy 55.88 135.89) (xy 55.88 138.43)
+			(xy 238.76 105.41) (xy 241.3 105.41)
 		)
 		(stroke
@@
 	(wire
 		(pts
-			(xy 238.76 100.33) (xy 241.3 100.33)
+			(xy 238.76 97.79) (xy 241.3 97.79)
 		)
 		(stroke
@@
 	(wire
 		(pts
-			(xy 238.76 97.79) (xy 241.3 97.79)
+			(xy 158.75 95.25) (xy 162.56 95.25)
 		)
 		(stroke
@@
 	(wire
 		(pts
-			(xy 158.75 95.25) (xy 162.56 95.25)
+			(xy 238.76 102.87) (xy 241.3 102.87)
 		)
 		(stroke
@@
 	(wire
 		(pts
-			(xy 254 100.33) (xy 256.54 100.33)
-		)
-		(stroke
-			(width 0)
-			(type default)
-		)
-	)
-	(wire
-		(pts
 			(xy 38.1 63.5) (xy 45.72 63.5)
 		)
@@
 	(wire
 		(pts
+			(xy 254 102.87) (xy 256.54 102.87)
+		)
+		(stroke
+			(width 0)
+			(type default)
+		)
+	)
+	(wire
+		(pts
+			(xy 238.76 100.33) (xy 241.3 100.33)
+		)
+		(stroke
+			(width 0)
+			(type default)
+		)
+	)
+	(wire
+		(pts
 			(xy 38.1 58.42) (xy 38.1 63.5)
 		)
@@
 	(wire
 		(pts
-			(xy 254 102.87) (xy 256.54 102.87)
-		)
-		(stroke
-			(width 0)
-			(type default)
-		)
-	)
-	(wire
-		(pts
 			(xy 254 115.57) (xy 256.54 115.57)
 		)
@@
 	(wire
 		(pts
-			(xy 238.76 105.41) (xy 241.3 105.41)
-		)
-		(stroke
-			(width 0)
-			(type default)
-		)
-	)
-	(wire
-		(pts
 			(xy 142.24 90.17) (xy 142.24 92.71)
 		)
@@
 	(global_label "PB1"
 		(shape input)
-		(at 238.76 100.33 180)
+		(at 256.54 100.33 0)
 		(fields_autoplaced yes)
 		(effects
@@
 				(size 1.27 1.27)
 			)
-			(justify right)
+			(justify left)
 		)
 		(property "Intersheetrefs" "${INTERSHEET_REFS}"
-			(at 232.0253 100.33 0)
+			(at 263.2747 100.33 0)
 			(effects
 				(font
 					(size 1.27 1.27)
 				)
-				(justify right)
+				(justify left)
 				(hide yes)
 			)
@@
 	(global_label "PA5"
 		(shape input)
-		(at 238.76 105.41 180)
+		(at 256.54 105.41 0)
 		(fields_autoplaced yes)
 		(effects
@@
 				(size 1.27 1.27)
 			)
-			(justify right)
+			(justify left)
 		)
 		(property "Intersheetrefs" "${INTERSHEET_REFS}"
-			(at 232.2067 105.41 0)
+			(at 263.0933 105.41 0)
 			(effects
 				(font
 					(size 1.27 1.27)
 				)
-				(justify right)
+				(justify left)
 				(hide yes)
 			)
@@
 	(global_label "PB2"
 		(shape input)
-		(at 256.54 100.33 0)
+		(at 238.76 100.33 180)
 		(fields_autoplaced yes)
 		(effects
@@
 				(size 1.27 1.27)
 			)
-			(justify left)
+			(justify right)
 		)
 		(property "Intersheetrefs" "${INTERSHEET_REFS}"
-			(at 263.2747 100.33 0)
+			(at 232.0253 100.33 0)
 			(effects
 				(font
 					(size 1.27 1.27)
 				)
-				(justify left)
+				(justify right)
 				(hide yes)
 			)
@@
 	(global_label "PA6"
 		(shape input)
-		(at 256.54 105.41 0)
+		(at 238.76 105.41 180)
 		(fields_autoplaced yes)
 		(effects
@@
 				(size 1.27 1.27)
 			)
-			(justify left)
+			(justify right)
 		)
 		(property "Intersheetrefs" "${INTERSHEET_REFS}"
-			(at 62.23 48.26 0)
+			(at 232.2067 105.41 0)
 			(effects
 				(font
 					(size 1.27 1.27)
 				)
+				(justify right)
 				(hide yes)
 			)
@@
 	(global_label "PB0"
 		(shape input)
-		(at 256.54 102.87 0)
+		(at 238.76 102.87 180)
 		(fields_autoplaced yes)
 		(effects
@@
 				(size 1.27 1.27)
 			)
-			(justify left)
+			(justify right)
 		)
 		(property "Intersheetrefs" "${INTERSHEET_REFS}"
-			(at 263.2747 102.87 0)
+			(at 232.0253 102.87 0)
 			(effects
 				(font
 					(size 1.27 1.27)
 				)
-				(justify left)
+				(justify right)
 				(hide yes)
 			)
@@
 	(global_label "PA7"
 		(shape input)
-		(at 238.76 102.87 180)
+		(at 256.54 102.87 0)
 		(fields_autoplaced yes)
 		(effects
@@
 				(size 1.27 1.27)
 			)
-			(justify right)
+			(justify left)
 		)
 		(property "Intersheetrefs" "${INTERSHEET_REFS}"
-			(at 232.2067 102.87 0)
+			(at 263.0933 102.87 0)
 			(effects
 				(font
 					(size 1.27 1.27)
 				)
-				(justify right)
+				(justify left)
 				(hide yes)
 			)
@@
 					(size 1.27 1.27)
 				)
+				(hide yes)
 			)
 		)
-		(property "Value" "~"
+		(property "Value" "DFLS140"
 			(at 58.42 127.6096 0)
 			(effects
@@
 			)
 		)
-		(property "Footprint" "Diode_SMD:D_SOD-123"
+		(property "Footprint" "Diode_SMD:D_PowerDI-123"
 			(at 58.42 130.81 0)
 			(effects
@@
 			)
 		)
-		(property "Value" "R_5.1K_0805"
+		(property "Value" "R_5.1K_0603"
 			(at 41.91 142.24 0)
 			(effects
@@
 			)
 		)
-		(property "Value" "R_5.1K_0805"
+		(property "Value" "R_5.1K_0603"
 			(at 41.91 144.78 0)
 			(effects
@@
 			)
 		)
-		(property "Value" "R_220_0805"
+		(property "Value" "R_220_0603"
 			(at 156.21 180.34 0)
 			(effects
@@
 			)
 		)
-		(property "Value" "R_220_0805"
+		(property "Value" "R_220_0603"
 			(at 170.18 180.34 0)
 			(effects
@@
 			)
 		)
-		(property "Display" "20pF"
+		(property "Display" "10pF"
 			(at 121.92 88.9 0)
 			(effects
@@
 			)
 		)
-		(property "Display" "20pF"
+		(property "Display" "10pF"
 			(at 142.24 88.9 0)
 			(effects
@@
 			)
 		)
-		(property "Value" "R_10K_0805"
+		(property "Value" "R_10K_0603"
 			(at 134.62 182.88 0)
 			(effects
@@
 			)
 		)
-		(property "Value" "R_10K_0805"
+		(property "Value" "R_10K_0603"
 			(at 114.3 167.64 0)
 			(effects
@@
 			)
 		)
-		(property "Footprint" "Crystal:Crystal_SMD_3225-4Pin_3.2x2.5mm"
+		(property "Footprint" "Crystal:Crystal_SMD_2016-4Pin_2.0x1.6mm"
 			(at 154.94 82.55 0)
 			(effects
@@
 			)
 		)
-		(property "Footprint" "Package_TO_SOT_SMD:SOT-323_SC-70"
+		(property "Footprint" "Package_TO_SOT_SMD:TSOT-23"
 			(at 37.465 95.885 0)
 			(effects
@@
 			)
 		)
-		(property "Value" "FB_0603"
+		(property "Value" "FB_0805"
 			(at 34.29 60.96 0)
 			(effects
@@
 			)
 		)
-		(property "Footprint" "Inductor_SMD:L_0603_1608Metric"
+		(property "Footprint" "Inductor_SMD:L_0805_2012Metric"
 			(at 39.37 57.15 0)
 			(effects
@@
 			)
 		)
-		(property "Value" "FB_0603"
+		(property "Value" "FB_0805"
 			(at 58.42 60.96 0)
 			(effects
@@
 			)
 		)
-		(property "Footprint" "Inductor_SMD:L_0603_1608Metric"
+		(property "Footprint" "Inductor_SMD:L_0805_2012Metric"
 			(at 63.5 57.15 0)
 			(effects

Commit message: pcb design update 1
Parts:
- C11, C12: value C_20PF_0603 -> C_10PF_0402; footprint Capacitor_SMD:C_0603_1608Metric -> Capacitor_SMD:C_0402_1005Metric
Changed lines of the file:
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@@
 			)
 		)
-		(property "Value" "C_20PF_0603"
+		(property "Value" "C_10PF_0402"
 			(at 123.19 90.17 0)
 			(effects
@@
 			)
 		)
-		(property "Footprint" "Capacitor_SMD:C_0603_1608Metric"
+		(property "Footprint" "Capacitor_SMD:C_0402_1005Metric"
 			(at 139.7 92.71 0)
 			(effects
@@
 			)
 		)
-		(property "Value" "C_20PF_0603"
+		(property "Value" "C_10PF_0402"
 			(at 143.51 90.17 0)
 			(effects
@@
 			)
 		)
-		(property "Footprint" "Capacitor_SMD:C_0603_1608Metric"
+		(property "Footprint" "Capacitor_SMD:C_0402_1005Metric"
 			(at 160.02 92.71 0)
 			(effects

Commit message: update new
Parts:
- C11, C12: value C_10PF_0402 -> C_10PF_0603; footprint Capacitor_SMD:C_0402_1005Metric -> Capacitor_SMD:C_0603_1608Metric
Changed lines of the file:
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@@
 			)
 		)
-		(property "Value" "C_10PF_0402"
+		(property "Value" "C_10PF_0603"
 			(at 123.19 90.17 0)
 			(effects
@@
 			)
 		)
-		(property "Footprint" "Capacitor_SMD:C_0402_1005Metric"
+		(property "Footprint" "Capacitor_SMD:C_0603_1608Metric"
 			(at 139.7 92.71 0)
 			(effects
@@
 			)
 		)
-		(property "Value" "C_10PF_0402"
+		(property "Value" "C_10PF_0603"
 			(at 143.51 90.17 0)
 			(effects
@@
 			)
 		)
-		(property "Footprint" "Capacitor_SMD:C_0402_1005Metric"
+		(property "Footprint" "Capacitor_SMD:C_0603_1608Metric"
 			(at 160.02 92.71 0)
 			(effects
